File: plain60-c.kicad_pcb (KiCad board)
At the start: 2 copper layers, 284.7 x 94.2 mm, 177 parts, among them J1 HRO-TYPE-C-31-M-12, J2 ISP, J3 ai03_ud, K1 KEYSW, K10 KEYSW, K11 KEYSW, K12 KEYSW, K13 KEYSW, K14 KEYSW, K15 KEYSW, K15-1 KEYSW, K16 KEYSW, K17 KEYSW, K18 KEYSW, K19 KEYSW, K2 KEYSW, K20 KEYSW, K21 KEYSW, K22 KEYSW, K23 KEYSW, K24 KEYSW, K25 KEYSW, K26 KEYSW, K27 KEYSW, K28 KEYSW, K29 KEYSW, K3 KEYSW, K31 KEYSW, K31-1 KEYSW, K32 KEYSW, K33 KEYSW, K34 KEYSW, K35 KEYSW, K36 KEYSW, K37 KEYSW, K38 KEYSW, K39 KEYSW, K4 KEYSW, K40 KEYSW, K41 KEYSW, K42 KEYSW, K43 KEYSW, K44 KEYSW, K44-1 KEYSW, K46 KEYSW, K46-1 KEYSW, K47 KEYSW, K48 KEYSW, K49 KEYSW, K5 KEYSW, K50 KEYSW, K51 KEYSW, K52 KEYSW, K53 KEYSW, K54 KEYSW, K55 KEYSW, K56 KEYSW, K57 KEYSW, K58 KEYSW, K58-1 KEYSW, K59 KEYSW, K6 KEYSW, K61 KEYSW, K61-1 KEYSW, K62 KEYSW, K62-1 KEYSW, K63 KEYSW, K63-1 KEYSW, K67 KEYSW, K67-1 KEYSW, K7 KEYSW, K71 KEYSW, K72 KEYSW, K72-1 KEYSW, K73 KEYSW, K73-1 KEYSW, K74 KEYSW, K74-1 KEYSW, K8 KEYSW, K9 KEYSW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

Commit message: add holes and move jst position
Parts:
- moved J3 70.5 mm to (5.08, 38.1), turned to 0 degrees
Routing:
- net D+: track 74.8 -> 56.9 mm
- net D-: track 71.9 -> 55.2 mm
- net VBUS: track 77.6 -> 69.3 mm
- net col14: track 257.3 -> 263.6 mm
- net col3: track 105.4 -> 106.6 mm
- added copper zone on F.Cu, net (none)
- removed copper zone on F.Cu, net GND
Other:
- outline, holes or cut-outs redrawn

Commit message: readme updated also added holes and shit
Parts:
- moved G*** 45.5 mm to (72.3, 38.3)
Other:
- board text added: "ZDC60 edition"
- board text added: "github.com/zd.collective/plain60-c"
- board text added: "https://github.com/zd-collective/plain60-c"
Changed lines of the file:
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@@
   )
   (module "Keeb_components:logo_new" locked (layer "B.Cu")
-    (at 26.789085 37.504719 180)
+    (at 72.31 38.3 180)
     (attr through_hole)
     (fp_text reference "G***" (at 0 0) (layer "B.SilkS") hide
@@
       (effects (font (size 1 1) (thickness 0.15)) (justify mirror))
     )
-    (fp_line (start -3.11 1.785) (end -2.06 1.785) (layer "B.SilkS") (width 0.12))
     (fp_line (start 3.11 -0.715) (end 3.11 1.785) (layer "B.SilkS") (width 0.12))
     (fp_line (start -1.94 -2.685) (end 1.94 -2.685) (layer "B.SilkS") (width 0.12))
+    (fp_line (start 3.11 1.785) (end 2.06 1.785) (layer "B.SilkS") (width 0.12))
+    (fp_line (start -3.11 1.785) (end -2.06 1.785) (layer "B.SilkS") (width 0.12))
     (fp_line (start -3.11 -0.715) (end -3.11 1.785) (layer "B.SilkS") (width 0.12))
     (fp_line (start -2.06 1.785) (end -2.06 2.775) (layer "B.SilkS") (width 0.12))
-    (fp_line (start 3.11 1.785) (end 2.06 1.785) (layer "B.SilkS") (width 0.12))
     (fp_line (start -3.9 -3.28) (end 3.9 -3.28) (layer "B.CrtYd") (width 0.05))
+    (fp_line (start 3.9 3.28) (end -3.9 3.28) (layer "B.CrtYd") (width 0.05))
     (fp_line (start -3.9 3.28) (end -3.9 -3.28) (layer "B.CrtYd") (width 0.05))
-    (fp_line (start 3.9 3.28) (end -3.9 3.28) (layer "B.CrtYd") (width 0.05))
     (fp_line (start 3.9 -3.28) (end 3.9 3.28) (layer "B.CrtYd") (width 0.05))
+    (fp_line (start -3 1.675) (end -3 -2.575) (layer "B.Fab") (width 0.1))
     (fp_line (start -1.5 0.967893) (end -1 1.675) (layer "B.Fab") (width 0.1))
+    (fp_line (start 3 1.675) (end 3 -2.575) (layer "B.Fab") (width 0.1))
+    (fp_line (start -3 -2.575) (end 3 -2.575) (layer "B.Fab") (width 0.1))
     (fp_line (start -2 1.675) (end -1.5 0.967893) (layer "B.Fab") (width 0.1))
-    (fp_line (start -3 1.675) (end -3 -2.575) (layer "B.Fab") (width 0.1))
-    (fp_line (start 3 1.675) (end 3 -2.575) (layer "B.Fab") (width 0.1))
     (fp_line (start -3 1.675) (end 3 1.675) (layer "B.Fab") (width 0.1))
-    (fp_line (start -3 -2.575) (end 3 -2.575) (layer "B.Fab") (width 0.1))
     (pad "1" smd roundrect (at -1.5 2.15) (size 0.6 1.85) (layers "B.Cu" "B.Paste" "B.Mask") (roundrect_rratio 0.25)
       (net 98 "VBUS") (pinfunction "Pin_1"))
@@
     (pad "4" smd roundrect (at 1.5 2.15) (size 0.6 1.85) (layers "B.Cu" "B.Paste" "B.Mask") (roundrect_rratio 0.25)
       (net 1 "GND") (pinfunction "Pin_4"))
+    (pad "MP" smd roundrect (at 3 -1.875) (size 1.6 1.8) (layers "B.Cu" "B.Paste" "B.Mask") (roundrect_rratio 0.208))
     (pad "MP" smd roundrect (at -3 -1.875) (size 1.6 1.8) (layers "B.Cu" "B.Paste" "B.Mask") (roundrect_rratio 0.208))
-    (pad "MP" smd roundrect (at 3 -1.875) (size 1.6 1.8) (layers "B.Cu" "B.Paste" "B.Mask") (roundrect_rratio 0.208))
-    (model "G:/Libraries/Keeb_components.pretty/models/SM04B-SRSS-TB.STEP"
+    (model "G:/Libraries/Keeb_components.pretty/models/SM04B-SRSS-TB.STEP" hide
       (offset (xyz 0 1.2 -0.3))
+      (scale (xyz 1 1 1))
+      (rotate (xyz 0 0 0))
+    )
+    (model "C:/random-keyboard-parts.pretty/JST-SR-4.step"
+      (offset (xyz 0 -2.8 0))
       (scale (xyz 1 1 1))
       (rotate (xyz -90 0 0))
@@
   (gr_circle (center 27.91 38.135) (end 30.16 38.135) (layer "Edge.Cuts") (width 0.2))
   (gr_circle (center 257.91 38.135) (end 260.16 38.135) (layer "Edge.Cuts") (width 0.2))
+  (gr_text "github.com/zd.collective/plain60-c" (at 72.35 58.1) (layer "F.Cu")
+    (effects (font (size 1.5 1.5) (thickness 0.3)))
+  )
   (gr_text "rev2.2" (at 47.62504 39.290658) (layer "B.SilkS")
     (effects (font (size 1 1) (thickness 0.15)) (justify mirror))
+  )
+  (gr_text "ZDC60 edition" (at 61.42 53.56) (layer "B.SilkS")
+    (effects (font (size 1.5 1.5) (thickness 0.3)) (justify mirror))
   )
   (gr_text "Plain60-C" (at 65.48443 36.909406) (layer "B.SilkS")
@@
     (effects (font (size 1 1) (thickness 0.15)) (justify mirror))
   )
+  (gr_text "https://github.com/zd-collective/plain60-c" (at 43.71 56.29) (layer "B.SilkS")
+    (effects (font (size 1.5 1.5) (thickness 0.3)) (justify mirror))
+  )
   (gr_text "Speaker\nAST1109MLTRQ\nPin B7" (at 163.711075 85.725072) (layer "B.SilkS")

Commit message: a
Routing:
- added copper zone on F.Cu, net GND
- removed copper zone on F.Cu, net (none)
Other:
- board text removed: "github.com/zd.collective/plain60-c"
Changed lines of the file:
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@@
   (gr_circle (center 27.91 38.135) (end 30.16 38.135) (layer "Edge.Cuts") (width 0.2))
   (gr_circle (center 257.91 38.135) (end 260.16 38.135) (layer "Edge.Cuts") (width 0.2))
-  (gr_text "github.com/zd.collective/plain60-c" (at 72.35 58.1) (layer "F.Cu")
-    (effects (font (size 1.5 1.5) (thickness 0.3)))
-  )
   (gr_text "rev2.2" (at 47.62504 39.290658) (layer "B.SilkS")
     (effects (font (size 1 1) (thickness 0.15)) (justify mirror))
@@
   (segment (start 95.059454 86.915698) (end 100.012584 86.915698) (width 0.25) (layer "B.Cu") (net 106))
   (segment (start 105.965714 87.435532) (end 104.554306 88.84694) (width 0.25) (layer "B.Cu") (net 106))
-  (zone (net 0) (net_name "") (layer "F.Cu") (hatch edge 0.508)
+  (zone (net 1) (net_name "GND") (layer "F.Cu") (hatch edge 0.508)
     (connect_pads (clearance 0.508))
     (min_thickness 0.254) (filled_areas_thickness no)
@@
     (polygon
       (pts
-        (xy 290.98 96.71)
-        (xy -6.24 98.7)
-        (xy -2.25 -2.59)
-        (xy -1.92 -2.59)
-        (xy 291.65 -4.91)
+        (xy 295.88 105.54)
+        (xy -9.01 109.97)
+        (xy -9.32 -9.9)
+        (xy 300.31 -12.75)
       )
     )
