File: plain60-c.kicad_pcb (KiCad board)
At the start: 2 copper layers, 284.7 x 94.2 mm, 165 parts, among them J2 ISP, J3 ai03_ud, K1 KEYSW, K10 KEYSW, K11 KEYSW, K12 KEYSW, K13 KEYSW, K14 KEYSW, K15 KEYSW, K15-1 KEYSW, K16 KEYSW, K17 KEYSW, K18 KEYSW, K19 KEYSW, K2 KEYSW, K20 KEYSW, K21 KEYSW, K22 KEYSW, K23 KEYSW, K24 KEYSW, K25 KEYSW, K26 KEYSW, K27 KEYSW, K28 KEYSW, K29 KEYSW, K3 KEYSW, K31 KEYSW, K31-1 KEYSW, K32 KEYSW, K33 KEYSW, K34 KEYSW, K35 KEYSW, K36 KEYSW, K37 KEYSW, K38 KEYSW, K39 KEYSW, K4 KEYSW, K40 KEYSW, K41 KEYSW, K42 KEYSW, K43 KEYSW, K44 KEYSW, K44-1 KEYSW, K46 KEYSW, K46-1 KEYSW, K47 KEYSW, K48 KEYSW, K49 KEYSW, K5 KEYSW, K50 KEYSW, K51 KEYSW, K52 KEYSW, K53 KEYSW, K54 KEYSW, K55 KEYSW, K56 KEYSW, K57 KEYSW, K58 KEYSW, K58-1 KEYSW, K59 KEYSW, K6 KEYSW, K61 KEYSW, K61-1 KEYSW, K62 KEYSW, K62-1 KEYSW, K63 KEYSW, K63-1 KEYSW, K67 KEYSW, K67-1 KEYSW, K7 KEYSW, K71 KEYSW, K72 KEYSW, K72-1 KEYSW, K73 KEYSW, K73-1 KEYSW, K74 KEYSW, K74-1 KEYSW, K8 KEYSW, K9 KEYSW, SW1 SW_PUSH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

Commit message: rounded traces and updated gerbers
Parts:
- removed the G*** at (170.3, 85.2)
- added G***: LOGO, weebSHit:noctus_mask, F.Cu at (171.8, 85.2)
Routing:
- net GND: track 50.2 -> 257.7 mm
- net Net-(R2-Pad2): track 167.4 -> 165.5 mm
- net VCC: track 280.1 -> 278.3 mm
- net Net-(R1-Pad1): track 164.0 -> 162.2 mm
- net row4: track 197.9 -> 196.9 mm
- net RST: track 140.8 -> 139.9 mm
- net Net-(D61-Pad2): track 36.5 -> 35.8 mm
- net col0: track 204.8 -> 204.2 mm
- removed copper zone on B.Cu, net GND
- removed copper zone on F.Cu, net GND
Other:
- board text added: "Noctus edition"
- board text removed: "Noctus ed."
